Commit message: base is now heavier and bigger, the robot doesnt tip anymore on spwan

File: install/main_nodes/share/main_nodes/urdf/base.urdf.xacro (robot description, xacro)
@@ -5,5 +5,5 @@
             <origin xyz="0 0 0.06" rpy="0 0 0"/>
             <geometry>
-                <box size="0.55 0.35 0.13" />
+                <box size="0.75 0.45 0.13" />
             </geometry>
         </visual>
@@ -16,5 +16,5 @@
         <inertial>
             <origin xyz="0 0 0.175" rpy="0 0 0"/>
-            <mass value="3.0"/>
+            <mass value="13.0"/>
             <inertia ixx="0.0502" ixy="0" ixz="0"
                      iyy="0.0502" iyz="0"
@@ -26,10 +26,10 @@
         <visual>
             <geometry>
-                <cylinder radius="0.07" length="0.035"/>
+                <cylinder radius="0.08" length="0.05"/>
             </geometry>
         </visual>
         <collision>
              <geometry>
-                <cylinder radius="0.07" length="0.035"/>
+                <cylinder radius="0.08" length="0.05"/>
             </geometry>
         </collision>
@@ -44,5 +44,5 @@
         <parent link="robot_base"/>
         <child link="left_wheel1"/>
-        <origin xyz="-0.15 0.18 0" rpy="-1.5707 0 0"/>
+        <origin xyz="-0.19 0.23 0" rpy="-1.5707 0 0"/>
         <axis xyz="0 0 1"/>
     </joint>
@@ -50,10 +50,10 @@
         <visual>
             <geometry>
-                <cylinder radius="0.07" length="0.035"/>
+                <cylinder radius="0.08" length="0.05"/>
             </geometry>
         </visual>
         <collision>
              <geometry>
-                <cylinder radius="0.07" length="0.035"/>
+                <cylinder radius="0.08" length="0.05"/>
             </geometry>
         </collision>
@@ -68,5 +68,5 @@
         <parent link="robot_base"/>
         <child link="left_wheel2"/>
-        <origin xyz="0.15 0.18 0" rpy="-1.5707 0 0"/>
+        <origin xyz="0.19 0.23 0" rpy="-1.5707 0 0"/>
         <axis xyz="0 0 1"/>
     </joint>
@@ -75,10 +75,10 @@
         <visual>
             <geometry>
-                <cylinder radius="0.07" length="0.035"/>
+                <cylinder radius="0.08" length="0.05"/>
             </geometry>
         </visual>
         <collision>
              <geometry>
-                <cylinder radius="0.07" length="0.035"/>
+                <cylinder radius="0.08" length="0.05"/>
             </geometry>
         </collision>
@@ -93,5 +93,5 @@
         <parent link="robot_base"/>
         <child link="right_wheel1"/>
-        <origin xyz="-0.15 -0.18 0" rpy="-1.5707 0 0"/>
+        <origin xyz="-0.19 -0.23 0" rpy="-1.5707 0 0"/>
         <axis xyz="0 0 1"/>
     </joint>
@@ -99,10 +99,10 @@
         <visual>
             <geometry>
-                <cylinder radius="0.07" length="0.035"/>
+                <cylinder radius="0.08" length="0.05"/>
             </geometry>
         </visual>
         <collision>
              <geometry>
-                <cylinder radius="0.07" length="0.035"/>
+                <cylinder radius="0.08" length="0.05"/>
             </geometry>
         </collision>
@@ -117,5 +117,5 @@
         <parent link="robot_base"/>
         <child link="right_wheel2"/>
-        <origin xyz="0.15 -0.18 0" rpy="-1.5707 0 0"/>
+        <origin xyz="0.19 -0.23 0" rpy="-1.5707 0 0"/>
         <axis xyz="0 0 1"/>
     </joint>

Commit message: okay now the teleop works after adjusting the inertia and gazebo properties to the new dimensions and masses, but there is a problem of tipping while moving

File: install/main_nodes/share/main_nodes/urdf/base.urdf.xacro (robot description, xacro)
@@ -8,16 +8,22 @@
             </geometry>
         </visual>
+        <!-- Collision must match the body so the robot rests on its WHEELS, not
+             on an oversized box. The old 0.28x0.28x0.35 box reached down to
+             z=-0.115 (below the wheels at -0.08), lifting the wheels off the
+             ground -> no traction -> robot couldn't drive. -->
         <collision>
             <origin xyz="0 0 0.06" rpy="0 0 0"/>
              <geometry>
-                <box size="0.28 0.28 0.35" />
+                <box size="0.75 0.45 0.13" />
             </geometry>
         </collision>
+        <!-- Inertia recomputed for a 13 kg, 0.75x0.45x0.13 box (I = m(a^2+b^2)/12);
+             COM lowered to z=0.04 (near the wheel axles) to resist tipping. -->
         <inertial>
-            <origin xyz="0 0 0.175" rpy="0 0 0"/>
+            <origin xyz="0 0 0.04" rpy="0 0 0"/>
             <mass value="13.0"/>
-            <inertia ixx="0.0502" ixy="0" ixz="0"
-                     iyy="0.0502" iyz="0"
-                     izz="0.0392"/>
+            <inertia ixx="0.2377" ixy="0" ixz="0"
+                     iyy="0.6277" iyz="0"
+                     izz="0.8288"/>
         </inertial>
     </link>
@@ -36,7 +42,7 @@
         <inertial>
             <mass value="0.3"/>
-            <inertia ixx="0.000211" ixy="0" ixz="0"
-                     iyy="0.000211" iyz="0"
-                     izz="0.00036"/>
+            <inertia ixx="0.0005425" ixy="0" ixz="0"
+                     iyy="0.0005425" iyz="0"
+                     izz="0.00096"/>
         </inertial>
     </link>
@@ -60,7 +66,7 @@
         <inertial>
             <mass value="0.3"/>
-            <inertia ixx="0.000211" ixy="0" ixz="0"
-                     iyy="0.000211" iyz="0"
-                     izz="0.00036"/>
+            <inertia ixx="0.0005425" ixy="0" ixz="0"
+                     iyy="0.0005425" iyz="0"
+                     izz="0.00096"/>
         </inertial>
     </link>
@@ -85,7 +91,7 @@
         <inertial>
             <mass value="0.3"/>
-            <inertia ixx="0.000211" ixy="0" ixz="0"
-                     iyy="0.000211" iyz="0"
-                     izz="0.00036"/>
+            <inertia ixx="0.0005425" ixy="0" ixz="0"
+                     iyy="0.0005425" iyz="0"
+                     izz="0.00096"/>
         </inertial>
     </link>
@@ -109,7 +115,7 @@
         <inertial>
             <mass value="0.3"/>
-            <inertia ixx="0.000211" ixy="0" ixz="0"
-                     iyy="0.000211" iyz="0"
-                     izz="0.00036"/>
+            <inertia ixx="0.0005425" ixy="0" ixz="0"
+                     iyy="0.0005425" iyz="0"
+                     izz="0.00096"/>
         </inertial>
     </link>
@@ -139,8 +145,8 @@
             <left_joint>left_wheel2_joint</left_joint>
             <right_joint>right_wheel2_joint</right_joint>
-            <wheel_separation>0.308</wheel_separation>
-            <wheel_separation>0.308</wheel_separation>
-            <wheel_diameter>0.098</wheel_diameter>
-            <wheel_diameter>0.098</wheel_diameter>
+            <wheel_separation>0.46</wheel_separation>
+            <wheel_separation>0.46</wheel_separation>
+            <wheel_diameter>0.16</wheel_diameter>
+            <wheel_diameter>0.16</wheel_diameter>
             <max_wheel_torque>20.0</max_wheel_torque>
             <max_wheel_acceleration>1.0</max_wheel_acceleration>

Commit message: increased frame size and wheel separation, now robot is stable while moving

File: install/main_nodes/share/main_nodes/urdf/base.urdf.xacro (robot description, xacro)
@@ -5,5 +5,5 @@
             <origin xyz="0 0 0.06" rpy="0 0 0"/>
             <geometry>
-                <box size="0.75 0.45 0.13" />
+                <box size="0.85 0.55 0.13" />
             </geometry>
         </visual>
@@ -15,15 +15,15 @@
             <origin xyz="0 0 0.06" rpy="0 0 0"/>
              <geometry>
-                <box size="0.75 0.45 0.13" />
+                <box size="0.85 0.55 0.13" />
             </geometry>
         </collision>
-        <!-- Inertia recomputed for a 13 kg, 0.75x0.45x0.13 box (I = m(a^2+b^2)/12);
+        <!-- Inertia recomputed for a 13 kg, 0.85x0.55x0.13 box (I = m(a^2+b^2)/12);
              COM lowered to z=0.04 (near the wheel axles) to resist tipping. -->
         <inertial>
             <origin xyz="0 0 0.04" rpy="0 0 0"/>
             <mass value="13.0"/>
-            <inertia ixx="0.2377" ixy="0" ixz="0"
-                     iyy="0.6277" iyz="0"
-                     izz="0.8288"/>
+            <inertia ixx="0.3460" ixy="0" ixz="0"
+                     iyy="0.8010" iyz="0"
+                     izz="1.1104"/>
         </inertial>
     </link>
@@ -50,5 +50,5 @@
         <parent link="robot_base"/>
         <child link="left_wheel1"/>
-        <origin xyz="-0.19 0.23 0" rpy="-1.5707 0 0"/>
+        <origin xyz="-0.3 0.27 0" rpy="-1.5707 0 0"/>
         <axis xyz="0 0 1"/>
     </joint>
@@ -74,5 +74,5 @@
         <parent link="robot_base"/>
         <child link="left_wheel2"/>
-        <origin xyz="0.19 0.23 0" rpy="-1.5707 0 0"/>
+        <origin xyz="0.3 0.27 0" rpy="-1.5707 0 0"/>
         <axis xyz="0 0 1"/>
     </joint>
@@ -99,5 +99,5 @@
         <parent link="robot_base"/>
         <child link="right_wheel1"/>
-        <origin xyz="-0.19 -0.23 0" rpy="-1.5707 0 0"/>
+        <origin xyz="-0.3 -0.27 0" rpy="-1.5707 0 0"/>
         <axis xyz="0 0 1"/>
     </joint>
@@ -123,5 +123,5 @@
         <parent link="robot_base"/>
         <child link="right_wheel2"/>
-        <origin xyz="0.19 -0.23 0" rpy="-1.5707 0 0"/>
+        <origin xyz="0.3 -0.27 0" rpy="-1.5707 0 0"/>
         <axis xyz="0 0 1"/>
     </joint>
@@ -145,6 +145,6 @@
             <left_joint>left_wheel2_joint</left_joint>
             <right_joint>right_wheel2_joint</right_joint>
-            <wheel_separation>0.46</wheel_separation>
-            <wheel_separation>0.46</wheel_separation>
+            <wheel_separation>0.54</wheel_separation>
+            <wheel_separation>0.54</wheel_separation>
             <wheel_diameter>0.16</wheel_diameter>
             <wheel_diameter>0.16</wheel_diameter>
