Commit message: added lidar link, placed between arm and diff drive base

File: install/main_nodes/share/main_nodes/urdf/robot.urdf.xacro (robot description, xacro)
@@ -3,8 +3,31 @@
 <xacro:include filename="$(find main_nodes)/urdf/base.urdf.xacro" />
 <xacro:include filename="$(find main_nodes)/urdf/arm.urdf.xacro" />
-<joint name="connector_joint" type="fixed">
+<link name="lidar_link">
+    <visual>
+        <geometry>
+            <cylinder radius="0.15" length="0.08"/>
+        </geometry>
+    </visual>
+    <collision>
+         <geometry>
+            <cylinder radius="0.15" length="0.08"/>
+        </geometry>
+    </collision>
+    <inertial>
+        <mass value="0.3"/>
+        <inertia ixx="0.0005425" ixy="0" ixz="0"
+                 iyy="0.0005425" iyz="0"
+                 izz="0.00096"/>
+    </inertial>
+</link>
+<joint name="lidar_joint" type="fixed">
     <parent link="robot_base"/>
-    <child link="arm_base_link"/>
+    <child link="lidar_link"/>
     <origin xyz="0 0 0.125" rpy="0 0 0"/>
 </joint>
+<joint name="connector_joint" type="fixed">
+    <parent link="lidar_link"/>
+    <child link="arm_base_link"/>
+    <origin xyz="0 0 0.04" rpy="0 0 0"/>
+</joint>
 </robot>
