Commit message: added gazebo lidar plugin and nav2 and slam yaml files, and new launch files for everything

File: install/main_nodes/share/main_nodes/urdf/arm.urdf.xacro (robot description, xacro)
@@ -1,387 +1 @@
-<?xml version="1.0" ?>
-<robot name="robot_arm" xmlns:xacro="http://www.ros.org/wiki/xacro">
-    <link name="arm_base_link">
-        <inertial>
-            <origin xyz="0 0 0.025" rpy="0 0 0"/>
-            <mass value="2.0"/>
-            <inertia ixx="0.007083" ixy="0" ixz="0" iyy="0.007083" iyz="0" izz="0.013333"/>
-        </inertial>
-        <visual>
-            <origin xyz="0 0 0.025" rpy="0 0 0"/>
-            <geometry>
-                <box size="0.2 0.2 0.05"/>
-            </geometry>
-            <material name="grey">
-                <color rgba="0.6 0.6 0.6 1.0"/>
-            </material>
-        </visual>
-        <collision>
-            <origin xyz="0 0 0.025" rpy="0 0 0"/>
-            <geometry>
-                <box size="0.18 0.18 0.04"/>
-            </geometry>
-        </collision>
-    </link>
-    <link name="waist_link">
-        <inertial>
-            <origin xyz="0 0 0" rpy="0 0 0"/>
-            <mass value="1.0"/>
-            <inertia ixx="0.002775" ixy="0" ixz="0" iyy="0.002775" iyz="0" izz="0.0018"/>
-        </inertial>
-        <visual>
-            <geometry>
-                <cylinder radius="0.06" length="0.15"/>
-            </geometry>
-            <material name="blue">
-                <color rgba="0.2 0.2 0.8 1.0"/>
-            </material>
-        </visual>
-        <collision>
-            <origin xyz="0 0 0" rpy="0 0 0"/>
-            <geometry>
-                <box size="0.09 0.09 0.13"/>
-            </geometry>
-        </collision>
-    </link>
-    <joint name="j1_waist" type="revolute">
-        <parent link="arm_base_link"/>
-        <child link="waist_link"/>
-        <origin xyz="0 0 0.12" rpy="0 0 0"/>
-        <axis xyz="0 0 1"/>
-        <limit lower="-3.14159" upper="3.14159" effort="100.0" velocity="1.0"/>
-    </joint>
-    <!-- J2 -->
-    <link name="shoulder_link">
-        <inertial>
-            <origin xyz="0 0 0" rpy="1.5708 0 1.5708"/>
-            <mass value="0.5"/>
-            <inertia ixx="0.0010167" ixy="0" ixz="0" iyy="0.0010167" iyz="0" izz="0.0004"/>
-        </inertial>
-        <visual>
-            <origin xyz="0 0 0" rpy="1.5708 0 1.5708"/>
-            <geometry>
-                <cylinder radius="0.04" length="0.14"/>
-            </geometry>
-            <material name="red">
-                <color rgba="0.8 0.2 0.2 1.0"/>
-            </material>
-        </visual>
-        <collision>
-            <origin xyz="0 0 0" rpy="1.5708 0 1.5708"/>
-            <geometry>
-                <box size="0.06 0.06 0.12"/>
-            </geometry>
-        </collision>
-    </link>
-    <joint name="j2_shoulder" type="revolute">
-        <parent link="waist_link"/>
-        <child link="shoulder_link"/>
-        <origin xyz="0.10 0 0.02" rpy="0 0 0"/>
-        <axis xyz="1 0 0"/>
-        <limit lower="-3.14159" upper="3.14159" effort="100.0" velocity="1.0"/>
-    </joint>
-    <link name="shoulder_arm">
-        <inertial>
-            <origin xyz="0 0 0" rpy="0 0 0"/>
-            <mass value="0.8"/>
-            <inertia ixx="0.008487" ixy="0" ixz="0" iyy="0.008487" iyz="0" izz="0.00064"/>
-        </inertial>
-        <visual>
-            <origin xyz="0 0 0" rpy="0 0 0"/>
-            <geometry>
-                <cylinder radius="0.04" length="0.35"/>
-            </geometry>
-            <material name="green">
-                <color rgba="0.2 0.8 0.2 1.0"/>
-            </material>
-        </visual>
-        <collision>
-            <origin xyz="0 0 0" rpy="0 0 0"/>
-            <geometry>
-                <box size="0.06 0.06 0.31"/>
-            </geometry>
-        </collision>
-    </link>
-    <joint name="a1_shoulder" type="fixed">
-        <parent link="shoulder_link"/>
-        <child link="shoulder_arm"/>
-        <origin xyz="0.027 0 0.18" rpy="0 0 0"/>
-    </joint>
-    <!-- J3 -->
-    <link name="elbow_link">
-        <inertial>
-            <origin xyz="0 0 0" rpy="1.5708 0 1.5708"/>
-            <mass value="0.5"/>
-            <inertia ixx="0.0012667" ixy="0" ixz="0" iyy="0.0012667" iyz="0" izz="0.0004"/>
-        </inertial>
-        <visual>
-            <origin xyz="0 0 0" rpy="1.5708 0 1.5708"/>
-            <geometry>
-                <cylinder radius="0.04" length="0.16"/>
-            </geometry>
-            <material name="red">
-                <color rgba="0.8 0.2 0.2 1.0"/>
-            </material>
-        </visual>
-        <collision>
-            <origin xyz="0 0 0" rpy="1.5708 0 1.5708"/>
-            <geometry>
-                <box size="0.06 0.06 0.14"/>
-            </geometry>
-        </collision>
-    </link>
-    <joint name="j3_elbow" type="revolute">
-        <parent link="shoulder_arm"/>
-        <child link="elbow_link"/>
-        <origin xyz="-0.09 0 0.134" rpy="0 0 0"/>
-        <axis xyz="1 0 0"/>
-        <limit lower="-3.14159" upper="3.14159" effort="100.0" velocity="1.0"/>
-    </joint>
-    <link name="elbow_arm">
-        <inertial>
-            <origin xyz="0 0 0" rpy="0 0 0"/>
-            <mass value="0.8"/>
-            <inertia ixx="0.008487" ixy="0" ixz="0" iyy="0.008487" iyz="0" izz="0.00064"/>
-        </inertial>
-        <visual>
-            <geometry>
-                <cylinder radius="0.04" length="0.35"/>
-            </geometry>
-            <material name="green">
-                <color rgba="0.2 0.8 0.2 1.0"/>
-            </material>
-        </visual>
-        <collision>
-            <origin xyz="0 0 0" rpy="0 0 0"/>
-            <geometry>
-                <box size="0.06 0.06 0.31"/>
-            </geometry>
-        </collision>
-    </link>
-     <joint name="a2_elbow" type="fixed">
-        <parent link="elbow_link"/>
-        <child link="elbow_arm"/>
-        <origin xyz="-0.04 0 0.18" rpy="0 0 0"/>
-    </joint>
-    <!-- J4 -->
-    <link name="wrist_link">
-        <inertial>
-            <origin xyz="0 0 0" rpy="0 0 0"/>
-            <mass value="0.3"/>
-            <inertia ixx="0.0001825" ixy="0" ixz="0" iyy="0.0001825" iyz="0" izz="0.00024"/>
-        </inertial>
-        <visual>
-            <geometry>
-                <cylinder radius="0.04" length="0.05"/>
-            </geometry>
-            <material name="blue">
-                <color rgba="0.2 0.2 0.8 1.0"/>
-            </material>
-        </visual>
-        <collision>
-            <origin xyz="0 0 0" rpy="0 0 0"/>
-            <geometry>
-                <box size="0.06 0.06 0.04"/>
-            </geometry>
-        </collision>
-    </link>
-    <joint name="j4_wrist" type="revolute">
-        <parent link="elbow_arm"/>
-        <child link="wrist_link"/>
-        <origin xyz="0 0 0.2" rpy="0 0 0"/>
-        <axis xyz="0 0 1"/>
-        <limit lower="-3.14159" upper="3.14159" effort="100.0" velocity="1.0"/>
-    </joint>
-    <!-- J5 -->
-    <link name="wrist_pitch_link">
-        <inertial>
-            <origin xyz="0 0 0" rpy="1.5708 0 1.5708"/>
-            <mass value="0.2"/>
-            <inertia ixx="0.00012667" ixy="0" ixz="0" iyy="0.00012667" iyz="0" izz="0.00004"/>
-        </inertial>
-        <visual>
-            <origin xyz="0 0 0" rpy="1.5708 0 1.5708"/>
-            <geometry>
-                <cylinder radius="0.02" length="0.08"/>
-            </geometry>
-            <material name="red">
-                <color rgba="0.8 0.2 0.2 1.0"/>
-            </material>
-        </visual>
-        <collision>
-            <origin xyz="0 0 0" rpy="1.5708 0 1.5708"/>
-            <geometry>
-                <box size="0.03 0.03 0.04"/>
-            </geometry>
-        </collision>
-    </link>
-    <joint name="j5_wrist" type="revolute">
-        <parent link="wrist_link"/>
-        <child link="wrist_pitch_link"/>
-        <origin xyz="0.06 0 0" rpy="0 0 0"/>
-        <axis xyz="1 0 0"/>
-        <limit lower="-3.14159" upper="3.14159" effort="100.0" velocity="1.0"/>
-    </joint>
-    <link name="wrist_arm">
-        <inertial>
-            <origin xyz="0 0 0" rpy="0 0 0"/>
-            <mass value="0.2"/>
-            <inertia ixx="0.00012667" ixy="0" ixz="0" iyy="0.00012667" iyz="0" izz="0.00004"/>
-        </inertial>
-        <visual>
-            <geometry>
-                <cylinder radius="0.02" length="0.08"/>
-            </geometry>
-            <material name="green">
-                <color rgba="0.2 0.8 0.2 1.0"/>
-            </material>
-        </visual>
-        <collision>
-            <origin xyz="0 0 0" rpy="0 0 0"/>
-            <geometry>
-                <box size="0.03 0.03 0.05"/>
-            </geometry>
-        </collision>
-    </link>
-     <joint name="a3_wrist" type="fixed">
-        <parent link="wrist_pitch_link"/>
-        <child link="wrist_arm"/>
-        <origin xyz="0.02 0 0.04" rpy="0 0 0"/>
-    </joint>
-    <!-- J6 -->
-     <link name="wrist_yaw_link">
-        <inertial>
-            <origin xyz="0 0 0" rpy="0 0 0"/>
-            <mass value="0.1"/>
-            <inertia ixx="0.000016" ixy="0" ixz="0" iyy="0.000016" iyz="0" izz="0.000016"/>
-        </inertial>
-        <visual>
-            <geometry>
-                <sphere radius="0.02"/>
-            </geometry>
-            <material name="purpel">
-                <color rgba="0.8 0.2 0.8 1.0"/>
-            </material>
-        </visual>
-        <collision>
-            <geometry>
-                <sphere radius="0.015"/>
-            </geometry>
-        </collision>
-    </link>
-    <joint name="j6_wrist" type="revolute">
-        <parent link="wrist_arm"/>
-        <child link="wrist_yaw_link"/>
-        <origin xyz="0 0 0.04" rpy="0 0 0"/>
-        <axis xyz="0 1 0"/>
-        <limit lower="-1.54159" upper="1.54159" effort="100.0" velocity="1.0"/>
-    </joint>
-    <!-- tool -->
-    <link name="tool_link">
-        <inertial>
-            <origin xyz="0 0 0" rpy="0 0 0"/>
-            <mass value="0.05"/>
-            <inertia ixx="0.00000792" ixy="0" ixz="0" iyy="0.00000792" iyz="0" izz="0.0000025"/>
-        </inertial>
-        <visual>
-            <geometry>
-                <cylinder radius="0.01" length="0.04"/>
-            </geometry>
-            <material name="else">
-                <color rgba="0.2 0.8 0.8 1.0"/>
-            </material>
-        </visual>
-        <collision>
-            <origin xyz="0 0 0" rpy="0 0 0"/>
-            <geometry>
-                <box size="0.015 0.015 0.03"/>
-            </geometry>
-        </collision>
-    </link>
-    <joint name="tool_joint" type="fixed">
-        <parent link="wrist_yaw_link"/>
-        <child link="tool_link"/>
-        <origin xyz="0 0 0.03" rpy="0 0 0"/>
-    </joint>
-     <link name="gripper_link">
-        <inertial>
-            <origin xyz="0 0 0" rpy="1.5708 0 0"/>
-            <mass value="0.05"/>
-            <inertia ixx="0.00001135" ixy="0" ixz="0" iyy="0.00001135" iyz="0" izz="0.000001875"/>
-        </inertial>
-        <visual>
-            <origin xyz="0 0 0" rpy="1.5708 0 0"/>
-            <geometry>
-                <box size="0.015 0.015 0.05"/>
-            </geometry>
-            <material name="else">
-                <color rgba="0.2 0.8 0.8 1.0"/>
-            </material>
-        </visual>
-        <collision>
-            <origin xyz="0 0 0" rpy="1.5708 0 0"/>
-            <geometry>
-                <box size="0.015 0.015 0.03"/>
-            </geometry>
-        </collision>
-    </link>
-    <joint name="gripper_joint" type="fixed">
-        <parent link="tool_link"/>
-        <child link="gripper_link"/>
-        <origin xyz="0 0 0.02" rpy="0 0 0"/>
-    </joint>
-    <link name="gripperfinger_left_link">
-        <inertial>
-            <origin xyz="0 0 0" rpy="0 0 0"/>
-            <mass value="0.02"/>
-            <inertia ixx="0.00000276" ixy="0" ixz="0" iyy="0.00000276" iyz="0" izz="0.0000001875"/>
-        </inertial>
-        <visual>
-            <geometry>
-                <box size="0.0075 0.0075 0.04"/>
-            </geometry>
-            <material name="else">
-                <color rgba="0.2 0.8 0.8 1.0"/>
-            </material>
-        </visual>
-        <collision>
-            <geometry>
-                <box size="0.0075 0.0075 0.04"/>
-            </geometry>
-        </collision>
-    </link>
-    <link name="gripperfinger_right_link">
-        <inertial>
-            <origin xyz="0 0 0" rpy="0 0 0"/>
-            <mass value="0.02"/>
-            <inertia ixx="0.00000276" ixy="0" ixz="0" iyy="0.00000276" iyz="0" izz="0.0000001875"/>
-        </inertial>
-        <visual>
-            <geometry>
-                <box size="0.0075 0.0075 0.04"/>
-            </geometry>
-            <material name="else">
-                <color rgba="0.2 0.8 0.8 1.0"/>
-            </material>
-        </visual>
-        <collision>
-            <geometry>
-                <box size="0.0075 0.0075 0.04"/>
-            </geometry>
-        </collision>
-    </link>
-    <joint name="gripperfinger_left_joint" type="prismatic">
-        <parent link="gripper_link"/>
-        <child link="gripperfinger_left_link"/>
-        <origin xyz="0 0.02 0.02" rpy="0 0 0"/>
-        <axis xyz="0 -1 0"/>
-        <limit lower="0" upper="0.02" effort="100.0" velocity="1.0"/>
-    </joint>
-    <joint name="gripperfinger_right_joint" type="prismatic">
-        <parent link="gripper_link"/>
-        <child link="gripperfinger_right_link"/>
-        <origin xyz="0 -0.02 0.02" rpy="0 0 0"/>
-        <axis xyz="0 1 0"/>
-        <limit lower="0" upper="0.02" effort="100.0" velocity="1.0"/>
-    </joint>
-</robot>
+/home/ibrahim/MobiArm/src/main_nodes/urdf/arm.urdf.xacro

File: install/main_nodes/share/main_nodes/urdf/base.urdf.xacro (robot description, xacro)
@@ -1,162 +1 @@
-<?xml version="1.0"?>
-<robot name="r2d2" xmlns:xacro="http://www.ros.org/wiki/xacro">
-    <link name="robot_base" >
-        <visual>
-            <origin xyz="0 0 0.06" rpy="0 0 0"/>
-            <geometry>
-                <box size="0.85 0.55 0.13" />
-            </geometry>
-        </visual>
-        <!-- Collision must match the body so the robot rests on its WHEELS, not
-             on an oversized box. The old 0.28x0.28x0.35 box reached down to
-             z=-0.115 (below the wheels at -0.08), lifting the wheels off the
-             ground -> no traction -> robot couldn't drive. -->
-        <collision>
-            <origin xyz="0 0 0.06" rpy="0 0 0"/>
-             <geometry>
-                <box size="0.85 0.55 0.13" />
-            </geometry>
-        </collision>
-        <!-- Inertia recomputed for a 13 kg, 0.85x0.55x0.13 box (I = m(a^2+b^2)/12);
-             COM lowered to z=0.04 (near the wheel axles) to resist tipping. -->
-        <inertial>
-            <origin xyz="0 0 0.04" rpy="0 0 0"/>
-            <mass value="13.0"/>
-            <inertia ixx="0.3460" ixy="0" ixz="0"
-                     iyy="0.8010" iyz="0"
-                     izz="1.1104"/>
-        </inertial>
-    </link>
-    <!-- left wheels -->
-    <link name="left_wheel1">
-        <visual>
-            <geometry>
-                <cylinder radius="0.08" length="0.05"/>
-            </geometry>
-        </visual>
-        <collision>
-             <geometry>
-                <cylinder radius="0.08" length="0.05"/>
-            </geometry>
-        </collision>
-        <inertial>
-            <mass value="0.3"/>
-            <inertia ixx="0.0005425" ixy="0" ixz="0"
-                     iyy="0.0005425" iyz="0"
-                     izz="0.00096"/>
-        </inertial>
-    </link>
-    <joint name="left_wheel1_joint" type="continuous">
-        <parent link="robot_base"/>
-        <child link="left_wheel1"/>
-        <origin xyz="-0.3 0.27 0" rpy="-1.5707 0 0"/>
-        <axis xyz="0 0 1"/>
-    </joint>
-    <link name="left_wheel2">
-        <visual>
-            <geometry>
-                <cylinder radius="0.08" length="0.05"/>
-            </geometry>
-        </visual>
-        <collision>
-             <geometry>
-                <cylinder radius="0.08" length="0.05"/>
-            </geometry>
-        </collision>
-        <inertial>
-            <mass value="0.3"/>
-            <inertia ixx="0.0005425" ixy="0" ixz="0"
-                     iyy="0.0005425" iyz="0"
-                     izz="0.00096"/>
-        </inertial>
-    </link>
-    <joint name="left_wheel2_joint" type="continuous">
-        <parent link="robot_base"/>
-        <child link="left_wheel2"/>
-        <origin xyz="0.3 0.27 0" rpy="-1.5707 0 0"/>
-        <axis xyz="0 0 1"/>
-    </joint>
-    <!-- right wheels -->
-    <link name="right_wheel1">
-        <visual>
-            <geometry>
-                <cylinder radius="0.08" length="0.05"/>
-            </geometry>
-        </visual>
-        <collision>
-             <geometry>
-                <cylinder radius="0.08" length="0.05"/>
-            </geometry>
-        </collision>
-        <inertial>
-            <mass value="0.3"/>
-            <inertia ixx="0.0005425" ixy="0" ixz="0"
-                     iyy="0.0005425" iyz="0"
-                     izz="0.00096"/>
-        </inertial>
-    </link>
-    <joint name="right_wheel1_joint" type="continuous">
-        <parent link="robot_base"/>
-        <child link="right_wheel1"/>
-        <origin xyz="-0.3 -0.27 0" rpy="-1.5707 0 0"/>
-        <axis xyz="0 0 1"/>
-    </joint>
-    <link name="right_wheel2">
-        <visual>
-            <geometry>
-                <cylinder radius="0.08" length="0.05"/>
-            </geometry>
-        </visual>
-        <collision>
-             <geometry>
-                <cylinder radius="0.08" length="0.05"/>
-            </geometry>
-        </collision>
-        <inertial>
-            <mass value="0.3"/>
-            <inertia ixx="0.0005425" ixy="0" ixz="0"
-                     iyy="0.0005425" iyz="0"
-                     izz="0.00096"/>
-        </inertial>
-    </link>
-    <joint name="right_wheel2_joint" type="continuous">
-        <parent link="robot_base"/>
-        <child link="right_wheel2"/>
-        <origin xyz="0.3 -0.27 0" rpy="-1.5707 0 0"/>
-        <axis xyz="0 0 1"/>
-    </joint>
-    <!-- wheel friction (helps the wheels grip the ground plane) -->
-    <gazebo reference="left_wheel1"><mu1>1.0</mu1><mu2>1.0</mu2></gazebo>
-    <gazebo reference="left_wheel2"><mu1>1.0</mu1><mu2>1.0</mu2></gazebo>
-    <gazebo reference="right_wheel1"><mu1>1.0</mu1><mu2>1.0</mu2></gazebo>
-    <gazebo reference="right_wheel2"><mu1>1.0</mu1><mu2>1.0</mu2></gazebo>
-    <!-- Differential drive controller (publishes /odom + odom->robot_base TF,
-         subscribes to /cmd_vel). Two wheel pairs driven together. -->
-    <gazebo>
-        <plugin name="diff_drive" filename="libgazebo_ros_diff_drive.so">
-            <ros>
-                <namespace>/</namespace>
-            </ros>
-            <num_wheel_pairs>2</num_wheel_pairs>
-            <!-- pair 1 -->
-            <left_joint>left_wheel1_joint</left_joint>
-            <right_joint>right_wheel1_joint</right_joint>
-            <!-- pair 2 -->
-            <left_joint>left_wheel2_joint</left_joint>
-            <right_joint>right_wheel2_joint</right_joint>
-            <wheel_separation>0.54</wheel_separation>
-            <wheel_separation>0.54</wheel_separation>
-            <wheel_diameter>0.16</wheel_diameter>
-            <wheel_diameter>0.16</wheel_diameter>
-            <max_wheel_torque>20.0</max_wheel_torque>
-            <max_wheel_acceleration>1.0</max_wheel_acceleration>
-            <command_topic>cmd_vel</command_topic>
-            <odometry_topic>odom</odometry_topic>
-            <odometry_frame>odom</odometry_frame>
-            <robot_base_frame>robot_base</robot_base_frame>
-            <publish_odom>true</publish_odom>
-            <publish_odom_tf>true</publish_odom_tf>
-            <publish_wheel_tf>true</publish_wheel_tf>
-        </plugin>
-    </gazebo>
-</robot>
+/home/ibrahim/MobiArm/src/main_nodes/urdf/base.urdf.xacro

File: install/main_nodes/share/main_nodes/urdf/robot.urdf.xacro (robot description, xacro)
@@ -1,33 +1 @@
-<?xml version="1.0"?>
-<robot name="mobiarm" xmlns:xacro="http://www.ros.org/wiki/xacro">
-<xacro:include filename="$(find main_nodes)/urdf/base.urdf.xacro" />
-<xacro:include filename="$(find main_nodes)/urdf/arm.urdf.xacro" />
-<link name="lidar_link">
-    <visual>
-        <geometry>
-            <cylinder radius="0.15" length="0.08"/>
-        </geometry>
-    </visual>
-    <collision>
-         <geometry>
-            <cylinder radius="0.15" length="0.08"/>
-        </geometry>
-    </collision>
-    <inertial>
-        <mass value="0.3"/>
-        <inertia ixx="0.0005425" ixy="0" ixz="0"
-                 iyy="0.0005425" iyz="0"
-                 izz="0.00096"/>
-    </inertial>
-</link>
-<joint name="lidar_joint" type="fixed">
-    <parent link="robot_base"/>
-    <child link="lidar_link"/>
-    <origin xyz="0 0 0.125" rpy="0 0 0"/>
-</joint>
-<joint name="connector_joint" type="fixed">
-    <parent link="lidar_link"/>
-    <child link="arm_base_link"/>
-    <origin xyz="0 0 0.04" rpy="0 0 0"/>
-</joint>
-</robot>
+/home/ibrahim/MobiArm/src/main_nodes/urdf/robot.urdf.xacro
