Commit message: added gazebo lidar plugin and nav2 and slam yaml files, and new launch files for everything

File: install/moveit_config/share/moveit_config/config/mobiarm.ros2_control.xacro (robot description, xacro)
@@ -1,66 +1 @@
-<?xml version="1.0"?>
-<robot xmlns:xacro="http://www.ros.org/wiki/xacro">
-    <xacro:macro name="mobiarm_ros2_control" params="name initial_positions_file use_gazebo:=false">
-        <xacro:property name="initial_positions" value="${load_yaml(initial_positions_file)['initial_positions']}"/>
-        <ros2_control name="${name}" type="system">
-            <hardware>
-                <xacro:if value="${use_gazebo}">
-                    <!-- Gazebo Classic: the controller_manager runs inside Gazebo -->
-                    <plugin>gazebo_ros2_control/GazeboSystem</plugin>
-                </xacro:if>
-                <xacro:unless value="${use_gazebo}">
-                    <!-- Mock hardware for the RViz-only demo (no physics) -->
-                    <plugin>mock_components/GenericSystem</plugin>
-                </xacro:unless>
-            </hardware>
-            <joint name="j1_waist">
-                <command_interface name="position"/>
-                <state_interface name="position">
-                  <param name="initial_value">${initial_positions['j1_waist']}</param>
-                </state_interface>
-            </joint>
-            <joint name="j2_shoulder">
-                <command_interface name="position"/>
-                <state_interface name="position">
-                  <param name="initial_value">${initial_positions['j2_shoulder']}</param>
-                </state_interface>
-            </joint>
-            <joint name="j3_elbow">
-                <command_interface name="position"/>
-                <state_interface name="position">
-                  <param name="initial_value">${initial_positions['j3_elbow']}</param>
-                </state_interface>
-            </joint>
-            <joint name="j4_wrist">
-                <command_interface name="position"/>
-                <state_interface name="position">
-                  <param name="initial_value">${initial_positions['j4_wrist']}</param>
-                </state_interface>
-            </joint>
-            <joint name="j5_wrist">
-                <command_interface name="position"/>
-                <state_interface name="position">
-                  <param name="initial_value">${initial_positions['j5_wrist']}</param>
-                </state_interface>
-            </joint>
-            <joint name="j6_wrist">
-                <command_interface name="position"/>
-                <state_interface name="position">
-                  <param name="initial_value">${initial_positions['j6_wrist']}</param>
-                </state_interface>
-            </joint>
-            <joint name="gripperfinger_left_joint">
-                <command_interface name="position"/>
-                <state_interface name="position">
-                  <param name="initial_value">${initial_positions['gripperfinger_left_joint']}</param>
-                </state_interface>
-            </joint>
-            <joint name="gripperfinger_right_joint">
-                <command_interface name="position"/>
-                <state_interface name="position">
-                  <param name="initial_value">${initial_positions['gripperfinger_right_joint']}</param>
-                </state_interface>
-            </joint>
-        </ros2_control>
-    </xacro:macro>
-</robot>
+/home/ibrahim/MobiArm/src/moveit_config/config/mobiarm.ros2_control.xacro

File: install/moveit_config/share/moveit_config/config/mobiarm.urdf.xacro (robot description, xacro)
@@ -1,24 +1 @@
-<?xml version="1.0"?>
-<robot xmlns:xacro="http://www.ros.org/wiki/xacro" name="mobiarm">
-    <xacro:arg name="initial_positions_file" default="initial_positions.yaml" />
-    <!-- Set to true when launching in Gazebo (see gazebo.launch.py). Leave false for the RViz demo. -->
-    <xacro:arg name="use_gazebo" default="false" />
-    <!-- Import mobiarm urdf file -->
-    <xacro:include filename="$(find main_nodes)/urdf/robot.urdf.xacro" />
-    <!-- Import control_xacro -->
-    <xacro:include filename="mobiarm.ros2_control.xacro" />
-    <xacro:mobiarm_ros2_control name="FakeSystem" initial_positions_file="$(arg initial_positions_file)" use_gazebo="$(arg use_gazebo)"/>
-    <!-- Gazebo-only: load the ros2_control plugin so the controller_manager runs
-         inside Gazebo for the arm + gripper joints.
-         NOTE: unlike BinPicking (a fixed-base arm), we deliberately do NOT anchor
-         robot_base to a `world` link. This is a mobile base: it must stay free to
-         drive via its diff-drive plugin and it rests on its wheels on the ground.
-         Pinning it to `world` would freeze the base and fight the diff-drive. -->
-    <xacro:if value="$(arg use_gazebo)">
-        <gazebo>
-            <plugin filename="libgazebo_ros2_control.so" name="gazebo_ros2_control">
-                <parameters>$(find moveit_config)/config/ros2_controllers.yaml</parameters>
-            </plugin>
-        </gazebo>
-    </xacro:if>
-</robot>
+/home/ibrahim/MobiArm/src/moveit_config/config/mobiarm.urdf.xacro

File: src/main_nodes/urdf/robot.urdf.xacro (robot description, xacro)
@@ -1,33 +1,61 @@
 <?xml version="1.0"?>
 <robot name="mobiarm" xmlns:xacro="http://www.ros.org/wiki/xacro">
-<xacro:include filename="$(find main_nodes)/urdf/base.urdf.xacro" />
-<xacro:include filename="$(find main_nodes)/urdf/arm.urdf.xacro" />
-<link name="lidar_link">
-    <visual>
-        <geometry>
-            <cylinder radius="0.15" length="0.08"/>
-        </geometry>
-    </visual>
-    <collision>
-         <geometry>
-            <cylinder radius="0.15" length="0.08"/>
-        </geometry>
-    </collision>
-    <inertial>
-        <mass value="0.3"/>
-        <inertia ixx="0.0005425" ixy="0" ixz="0"
-                 iyy="0.0005425" iyz="0"
-                 izz="0.00096"/>
-    </inertial>
-</link>
-<joint name="lidar_joint" type="fixed">
-    <parent link="robot_base"/>
-    <child link="lidar_link"/>
-    <origin xyz="0 0 0.125" rpy="0 0 0"/>
-</joint>
-<joint name="connector_joint" type="fixed">
-    <parent link="lidar_link"/>
-    <child link="arm_base_link"/>
-    <origin xyz="0 0 0.04" rpy="0 0 0"/>
-</joint>
+    <xacro:include filename="$(find main_nodes)/urdf/base.urdf.xacro" />
+    <xacro:include filename="$(find main_nodes)/urdf/arm.urdf.xacro" />
+    <link name="lidar_link">
+        <visual>
+            <geometry>
+                <cylinder radius="0.15" length="0.08"/>
+            </geometry>
+        </visual>
+        <collision>
+            <geometry>
+                <cylinder radius="0.15" length="0.08"/>
+            </geometry>
+        </collision>
+        <inertial>
+            <mass value="0.3"/>
+            <inertia ixx="0.0005425" ixy="0" ixz="0"
+                    iyy="0.0005425" iyz="0"
+                    izz="0.00096"/>
+        </inertial>
+    </link>
+    <joint name="lidar_joint" type="fixed">
+        <parent link="robot_base"/>
+        <child link="lidar_link"/>
+        <origin xyz="0 0 0.125" rpy="0 0 0"/>
+    </joint>
+    <joint name="connector_joint" type="fixed">
+        <parent link="lidar_link"/>
+        <child link="arm_base_link"/>
+        <origin xyz="0 0 0.04" rpy="0 0 0"/>
+    </joint>
+    <gazebo reference="lidar_link">
+        <sensor type="ray" name="lidar">
+            <pose>0 0 0 0 0 0</pose>
+            <always_on>true</always_on>
+            <visualize>true</visualize>
+            <update_rate>10</update_rate>
+            <ray>
+            <scan>
+                <horizontal>
+                <samples>360</samples>
+                <min_angle>-3.14159</min_angle>
+                <max_angle>3.14159</max_angle>
+                </horizontal>
+            </scan>
+            <range>
+                <min>0.15</min>
+                <max>12.0</max>
+            </range>
+            </ray>
+            <plugin name="lidar_plugin" filename="libgazebo_ros_ray_sensor.so">
+            <ros>
+                <remapping>~/out:=scan</remapping>
+            </ros>
+            <output_type>sensor_msgs/LaserScan</output_type>
+            <frame_name>lidar_link</frame_name>
+            </plugin>
+        </sensor>
+    </gazebo>
 </robot>
