Commit message: fixed slef scan by lidar rays by lifting the pose of the lidar

File: src/main_nodes/urdf/robot.urdf.xacro (robot description, xacro)
@@ -6,10 +6,10 @@
         <visual>
             <geometry>
-                <cylinder radius="0.15" length="0.08"/>
+                <cylinder radius="0.15" length="0.05"/>
             </geometry>
         </visual>
         <collision>
             <geometry>
-                <cylinder radius="0.15" length="0.08"/>
+                <cylinder radius="0.15" length="0.05"/>
             </geometry>
         </collision>
@@ -24,14 +24,18 @@
         <parent link="robot_base"/>
         <child link="lidar_link"/>
-        <origin xyz="0 0 0.125" rpy="0 0 0"/>
+        <origin xyz="0 0 0.15" rpy="0 0 0"/>
     </joint>
     <joint name="connector_joint" type="fixed">
         <parent link="lidar_link"/>
         <child link="arm_base_link"/>
-        <origin xyz="0 0 0.04" rpy="0 0 0"/>
+        <origin xyz="0 0 0.025" rpy="0 0 0"/>
     </joint>
     <gazebo reference="lidar_link">
         <sensor type="ray" name="lidar">
-            <pose>0 0 0 0 0 0</pose>
+            <!-- Raise the scan plane 2 cm above lidar_link's origin so it sits in
+                 the 4 cm gap between the base top (z=0.125) and the arm base bottom
+                 (z=0.165). At z=0 the plane grazed the base top and the lidar saw
+                 its own chassis as a ring of phantom obstacles. -->
+            <pose>0 0 0.02 0 0 0</pose>
             <always_on>true</always_on>
             <visualize>true</visualize>

Commit message: fixed lidar rays collision, with removing the collision tag on the lidar link. since it was ultering the radar scan

File: src/main_nodes/urdf/robot.urdf.xacro (robot description, xacro)
@@ -9,9 +9,11 @@
             </geometry>
         </visual>
-        <collision>
-            <geometry>
-                <cylinder radius="0.15" length="0.05"/>
-            </geometry>
-        </collision>
+        <!-- NO collision on purpose. The ray sensor is mounted at this link's
+             origin, and range_min (0.15) equals the old collision cylinder's
+             radius (0.15) -> every beam terminated on its own housing at 0.15 m,
+             got clipped as out-of-range, and returned inf. Result: the lidar was
+             blind (it saw neither the walls nor the table). lidar_link is a rigid
+             connector between base and arm (all fixed joints = one rigid body),
+             so it needs no collision of its own. -->
         <inertial>
             <mass value="0.3"/>
@@ -33,8 +35,8 @@
     <gazebo reference="lidar_link">
         <sensor type="ray" name="lidar">
-            <!-- Raise the scan plane 2 cm above lidar_link's origin so it sits in
-                 the 4 cm gap between the base top (z=0.125) and the arm base bottom
-                 (z=0.165). At z=0 the plane grazed the base top and the lidar saw
-                 its own chassis as a ring of phantom obstacles. -->
+            <!-- Scan plane 2 cm above lidar_link's origin: with lidar_joint at
+                 z=0.15 (robot_base frame) this puts the beam at z~0.17, clearing
+                 the base top (z=0.125) and staying under the arm base collision
+                 (starts ~z=0.18). -->
             <pose>0 0 0.02 0 0 0</pose>
             <always_on>true</always_on>

Commit message: added depth camera and its stand, but problem with self lidar collision

File: src/main_nodes/urdf/robot.urdf.xacro (robot description, xacro)
@@ -65,3 +65,77 @@
         </sensor>
     </gazebo>
+    <link name="camera_link">
+        <visual>
+            <geometry>
+                <box size="0.05 0.1 0.05"/>
+            </geometry>
+        </visual>
+        <collision>
+            <geometry><box size="0.05 0.05 0.05" /></geometry>
+        </collision>
+        <inertial>
+            <mass value="0.3"/>
+            <inertia ixx="0.0005425" ixy="0" ixz="0"
+                    iyy="0.0005425" iyz="0"
+                    izz="0.00096"/>
+        </inertial>
+    </link>
+    <link name="camera_optical_frame"/>
+    <joint name="camera_optical_joint" type="fixed">
+        <parent link="camera_link"/>
+        <child link="camera_optical_frame"/>
+        <origin xyz="0 0 0" rpy="-1.5708 0 -1.5708"/>
+    </joint>
+    <link name="camera_stand_link">
+        <visual>
+            <geometry>
+                <cylinder radius="0.025" length="0.1"/>
+            </geometry>
+        </visual>
+        <collision>
+            <geometry><cylinder radius="0.025" length="0.1"/></geometry>
+        </collision>
+        <inertial>
+            <mass value="0.3"/>
+            <inertia ixx="0.0005425" ixy="0" ixz="0"
+                    iyy="0.0005425" iyz="0"
+                    izz="0.00096"/>
+        </inertial>
+    </link>
+    <joint name="camera_stand_joint" type="fixed">
+        <parent link="robot_base"/>
+        <child link="camera_stand_link"/>
+        <origin xyz="0.4 0 0.17" rpy="0 0 0"/>
+    </joint>
+    <joint name="camera_joint" type="fixed">
+        <parent link="camera_stand_link"/>
+        <child link="camera_link"/>
+        <origin xyz="0 0 0.05" rpy="0 0 0"/>
+    </joint>
+    <gazebo reference="camera_link">
+        <sensor name="camera" type="depth">
+            <always_on>true</always_on>
+            <update_rate>30</update_rate>
+            <visualize>true</visualize>
+            <camera>
+                <horizontal_fov>1.047</horizontal_fov>   <!-- ~60 degrees -->
+                <image>
+                    <width>640</width>
+                    <height>480</height>
+                    <format>R8G8B8</format>
+                </image>
+                <clip>
+                    <near>0.05</near>
+                    <far>10.0</far>
+                </clip>
+            </camera>
+            <plugin name="camera_plugin" filename="libgazebo_ros_camera.so">
+                <camera_name>camera</camera_name>
+                <frame_name>camera_optical_frame</frame_name>
+                <!-- valid depth range; readings outside come back as NaN -->
+                <min_depth>0.05</min_depth>
+                <max_depth>10.0</max_depth>
+            </plugin>
+        </sensor>
+    </gazebo>
 </robot>

Commit message: added inertia tag for the imu

File: src/main_nodes/urdf/robot.urdf.xacro (robot description, xacro)
@@ -148,7 +148,18 @@
         </sensor>
     </gazebo>
-    <link name="imu_link"/>
-        <joint name="imu_joint" type="fixed">
-        <parent link="robot_base"/><child link="imu_link"/>
+    <!-- imu_link needs an <inertial> block: Gazebo Classic lumps a MASSLESS
+         fixed-joint child into its parent and drops the link, taking the
+         <gazebo reference="imu_link"> sensor with it -> /imu never publishes and
+         the EKF silently runs wheel-only (same yaw drift). A tiny mass keeps the
+         link (and its IMU sensor) alive, exactly like lidar_link/camera_link. -->
+    <link name="imu_link">
+        <inertial>
+            <mass value="0.01"/>
+            <inertia ixx="1e-6" ixy="0" ixz="0" iyy="1e-6" iyz="0" izz="1e-6"/>
+        </inertial>
+    </link>
+    <joint name="imu_joint" type="fixed">
+        <parent link="robot_base"/>
+        <child link="imu_link"/>
         <origin xyz="0 0 0.05" rpy="0 0 0"/>
     </joint>
