Commit message: added imu sensor and ekf config, now the robot tf or pos is fetched through the fused ekf which has a perfect yaw accuracy + the old vx accuracy from the diff drive plugin on odom

File: src/main_nodes/urdf/base.urdf.xacro (robot description, xacro)
@@ -156,5 +156,5 @@
             <robot_base_frame>robot_base</robot_base_frame>
             <publish_odom>true</publish_odom>
-            <publish_odom_tf>true</publish_odom_tf>
+            <publish_odom_tf>false</publish_odom_tf>
             <publish_wheel_tf>true</publish_wheel_tf>
         </plugin>

File: src/main_nodes/urdf/robot.urdf.xacro (robot description, xacro)
@@ -148,3 +148,17 @@
         </sensor>
     </gazebo>
+    <link name="imu_link"/>
+        <joint name="imu_joint" type="fixed">
+        <parent link="robot_base"/><child link="imu_link"/>
+        <origin xyz="0 0 0.05" rpy="0 0 0"/>
+    </joint>
+    <gazebo reference="imu_link">
+    <sensor name="imu_sensor" type="imu">
+        <always_on>true</always_on><update_rate>100</update_rate>
+        <plugin name="imu_plugin" filename="libgazebo_ros_imu_sensor.so">
+        <ros><remapping>~/out:=imu</remapping></ros>
+        <frame_name>imu_link</frame_name>
+        </plugin>
+    </sensor>
+    </gazebo>
 </robot>

Commit message: removed all traces of the imu and ekf

File: src/main_nodes/urdf/base.urdf.xacro (robot description, xacro)
@@ -163,8 +163,9 @@
             <robot_base_frame>robot_base</robot_base_frame>
             <publish_odom>true</publish_odom>
-            <!-- DIAGNOSTIC A/B: set back to true so the plugin publishes odom->robot_base
-                 itself (pure wheel odometry, pre-EKF behaviour). MUST disable the ekf_node
-                 in nav2_slam.launch.py at the same time, or two nodes publish the same TF
-                 and fight. Set back to false + re-enable EKF to restore the fused setup. -->
+            <!-- The diff-drive plugin publishes odom->robot_base directly from wheel
+                 odometry. An EKF/IMU fusion used to own this TF, but it introduced a
+                 yaw-dependent map/scan shift during turns (the scans swung in the odom
+                 frame as the robot rotated), so odom->base is sourced purely from the
+                 plugin. SLAM's map->odom absorbs the residual wheel-odometry drift. -->
             <publish_odom_tf>true</publish_odom_tf>
             <publish_wheel_tf>true</publish_wheel_tf>

File: src/main_nodes/urdf/robot.urdf.xacro (robot description, xacro)
@@ -148,28 +148,3 @@
         </sensor>
     </gazebo>
-    <!-- imu_link needs an <inertial> block: Gazebo Classic lumps a MASSLESS
-         fixed-joint child into its parent and drops the link, taking the
-         <gazebo reference="imu_link"> sensor with it -> /imu never publishes and
-         the EKF silently runs wheel-only (same yaw drift). A tiny mass keeps the
-         link (and its IMU sensor) alive, exactly like lidar_link/camera_link. -->
-    <link name="imu_link">
-        <inertial>
-            <mass value="0.01"/>
-            <inertia ixx="1e-6" ixy="0" ixz="0" iyy="1e-6" iyz="0" izz="1e-6"/>
-        </inertial>
-    </link>
-    <joint name="imu_joint" type="fixed">
-        <parent link="robot_base"/>
-        <child link="imu_link"/>
-        <origin xyz="0 0 0.05" rpy="0 0 0"/>
-    </joint>
-    <gazebo reference="imu_link">
-    <sensor name="imu_sensor" type="imu">
-        <always_on>true</always_on><update_rate>100</update_rate>
-        <plugin name="imu_plugin" filename="libgazebo_ros_imu_sensor.so">
-        <ros><remapping>~/out:=imu</remapping></ros>
-        <frame_name>imu_link</frame_name>
-        </plugin>
-    </sensor>
-    </gazebo>
 </robot>

Commit message: added gitignore and changed colors of base components

File: src/main_nodes/urdf/base.urdf.xacro (robot description, xacro)
@@ -7,4 +7,7 @@
                 <box size="0.85 0.55 0.13" />
             </geometry>
+            <material name="body_orange">
+                <color rgba="0.9 0.45 0.05 1.0"/>
+            </material>
         </visual>
         <!-- Collision matches the body so the robot rests on its wheels; an
@@ -30,4 +33,7 @@
                 <cylinder radius="0.08" length="0.05"/>
             </geometry>
+            <material name="wheel_black">
+                <color rgba="0.12 0.12 0.12 1.0"/>
+            </material>
         </visual>
         <collision>
@@ -54,4 +60,7 @@
                 <cylinder radius="0.08" length="0.05"/>
             </geometry>
+            <material name="wheel_black">
+                <color rgba="0.12 0.12 0.12 1.0"/>
+            </material>
         </visual>
         <collision>
@@ -78,4 +87,7 @@
                 <cylinder radius="0.08" length="0.05"/>
             </geometry>
+            <material name="wheel_black">
+                <color rgba="0.12 0.12 0.12 1.0"/>
+            </material>
         </visual>
         <collision>
@@ -102,4 +114,7 @@
                 <cylinder radius="0.08" length="0.05"/>
             </geometry>
+            <material name="wheel_black">
+                <color rgba="0.12 0.12 0.12 1.0"/>
+            </material>
         </visual>
         <collision>
@@ -124,8 +139,11 @@
          traction); mu2 low so wheels scrub sideways and the base can yaw (mu2=1
          pinned them laterally -> ~11% of commanded rotation). -->
-    <gazebo reference="left_wheel1"><mu1>1.0</mu1><mu2>0.7</mu2><fdir1>1 0 0</fdir1></gazebo>
-    <gazebo reference="left_wheel2"><mu1>1.0</mu1><mu2>0.7</mu2><fdir1>1 0 0</fdir1></gazebo>
-    <gazebo reference="right_wheel1"><mu1>1.0</mu1><mu2>0.7</mu2><fdir1>1 0 0</fdir1></gazebo>
-    <gazebo reference="right_wheel2"><mu1>1.0</mu1><mu2>0.7</mu2><fdir1>1 0 0</fdir1></gazebo>
+    <!-- Gazebo ignores the URDF <material> above (that only colours RViz), so the
+         render colour has to be repeated here per link. -->
+    <gazebo reference="left_wheel1"><mu1>1.0</mu1><mu2>0.7</mu2><fdir1>1 0 0</fdir1><material>Gazebo/Black</material></gazebo>
+    <gazebo reference="left_wheel2"><mu1>1.0</mu1><mu2>0.7</mu2><fdir1>1 0 0</fdir1><material>Gazebo/Black</material></gazebo>
+    <gazebo reference="right_wheel1"><mu1>1.0</mu1><mu2>0.7</mu2><fdir1>1 0 0</fdir1><material>Gazebo/Black</material></gazebo>
+    <gazebo reference="right_wheel2"><mu1>1.0</mu1><mu2>0.7</mu2><fdir1>1 0 0</fdir1><material>Gazebo/Black</material></gazebo>
+    <gazebo reference="robot_base"><material>Gazebo/Orange</material></gazebo>
     <!-- Differential drive: publishes /odom + odom->robot_base TF, subscribes /cmd_vel. -->
     <gazebo>

File: src/main_nodes/urdf/robot.urdf.xacro (robot description, xacro)
@@ -66,4 +66,7 @@
                 <box size="0.05 0.1 0.05"/>
             </geometry>
+            <material name="sensor_turquoise">
+                <color rgba="0.1 0.65 0.6 1.0"/>
+            </material>
         </visual>
         <!-- Collision kept (honest sim): the real lidar hits this; self-hits are
@@ -90,4 +93,7 @@
                 <cylinder radius="0.025" length="0.1"/>
             </geometry>
+            <material name="sensor_turquoise">
+                <color rgba="0.1 0.65 0.6 1.0"/>
+            </material>
         </visual>
         <!-- Collision kept (see camera_link): crosses the scan plane; self-hits
@@ -113,5 +119,8 @@
         <origin xyz="0 0 0.05" rpy="0 0 0"/>
     </joint>
+    <!-- Stand + camera share one colour so they read as a single mast. -->
+    <gazebo reference="camera_stand_link"><material>Gazebo/Turquoise</material></gazebo>
     <gazebo reference="camera_link">
+        <material>Gazebo/Turquoise</material>
         <sensor name="camera" type="depth">
             <always_on>true</always_on>
